File: electronics/CPU.sch (KiCad schematic (older format))
At the start: 4 parts

Commit message: Added isolators, updated CPU pins
Parts:
- added C? (x6): 0.1uF, symbol Device:C
- added J?: FTSH-105-XX-X-DV, SAMTEC_FTSH-105-XX-X-DV, symbol FTSH-105-XX-X-DV:FTSH-105-XX-X-DV
- added U? (x2): MAX14930DASE+, 21-0041_S16+1_MXM, symbol MAX14930DASE+:MAX14930DASE+
- added U?: MAX12930EASA+, 21-0041B_8_MXM, symbol MAX12930EASA:MAX12930EASA+
Connections:
- net labels added: +3V3, +5VD, CPU_SWCLK, CPU_SWDIO, Earth, MCU-MOT1en1, MCU-MOT1en2, MCU-MOT2en1, MCU-MOT2en2, MCU-MOT3en1, MCU-MOT3en2, MCU-TRW_PWM, MCU-mot_off, MCU-mot_sleep, MCU_NRST, MOT1en_1, MOT1en_2, MOT2en_1, MOT2en_2, MOT3en_1, MOT3en_2, MOT_off, MOT_sleep, TRW_PWM
- net labels removed: VCC
- wire segments 10 -> 70
Other:
- moved on the sheet: C?, U?

Commit message: Added connectors, started relabeling pins
Parts:
- removed C? (x2): 0.1uF, symbol Device:C
- removed J?: FTSH-105-XX-X-DV, SAMTEC_FTSH-105-XX-X-DV, symbol FTSH-105-XX-X-DV:FTSH-105-XX-X-DV
- removed U?: MAX12930EASA+, 21-0041B_8_MXM, symbol MAX12930EASA:MAX12930EASA+
- added C? (x2): 0.1uF, symbol Device:C
- added U?: MAX14930DASE+, 21-0041_S16+1_MXM, symbol MAX14930DASE+:MAX14930DASE+
Connections:
- net labels added: Aim-serv_PWM, Hold-serv_PWM, MCU-Aim-serv_PWM, MCU-Hold-serv_PWM
- net labels removed: CPU_SWCLK, CPU_SWDIO, MCU_NRST
- wire segments 70 -> 72
