File: electronics/Voltage regulator.sch (KiCad schematic (older format))
At the start: 10 parts

Commit message: Another restructure, added CPU pins, updated V regulators
Parts:
- removed C? (x4): 1uF, symbol Device:C
- removed C?: CP, symbol Device:CP
- removed J? (x2): 3mm_pad, symbol Electronics:3mm_pad
- removed J?: 10118193-0001LF, FCI_10118193-0001LF, symbol 10118193-0001LF:10118193-0001LF
- removed U?: NCP164, symbol Electronics:NCP164
- removed U?: NCV8730, symbol Electronics:NCV8730
Connections:
- net labels removed: +3V3, +5VD, +5VL, Earth, GND, Vdrive
- wire segments 8 -> 0
Other:
- note removed: "Battery connection pads"
- note removed: "Battery to driver logic 5V"
- note removed: "USB 5V to CPU logic 3v3"
- note removed: "USB port"
