File: electronics/Connectors.sch (KiCad schematic (older format))
At the start: 1 part

Commit message: Another restructure, added CPU pins, updated V regulators
Parts:
- added C?: 4.7uF, symbol Device:CP
- added C?: 33uF, symbol Device:C
- added C?: 0.47uF, symbol Device:C
- added C? (x5): 0.1uF, symbol Device:C
- added C? (x2): 10uF, symbol Device:C
- added D?: RED_LED, symbol Device:LED
- added J? (x6): 215079-4, TE_215079-4, symbol 215079-4:215079-4
- added J?: 10118193-0001LF, FCI_10118193-0001LF, symbol 10118193-0001LF:10118193-0001LF
- added J? (x2): 3mm_pad, symbol Electronics:3mm_pad
- added L?: 5.6uH, symbol Device:L
- added R?: 30Ohm, symbol Device:R
- added R?: 10KOhm, symbol Device:R
- added R?: 52.3KOhm, symbol Device:R
- added R?: 3.3KOhm, symbol Device:R
- added U?: TPS56339DDC, Package_TO_SOT_SMD:SOT-23-6, symbol Regulator_Switching:TPS56339DDC
- added U?: LM3940IT-3.3, TO254P1054X470X1955-3, symbol LM3940IT-3.3:LM3940IT-3.3
Connections:
- net labels added: +5VD, +5VL, Aim-serv_PWM, Earth, Hold-serv_PWM, MCU-USB_DM, MCU-USB_DP, MCU-mot1-enc_1, MCU-mot1-enc_2, MCU-mot2-enc_1, MCU-mot2-enc_2, MCU-mot3-enc_1, MCU-mot3-enc_2, MCU_SWCLK, MCU_SWDIO, TRW_PWM, Vdrive
- net labels removed: CPU_SWCLK, CPU_SWDIO
- wire segments 11 -> 49
- no-connect marks 0 -> 1
Other:
- note added: "Aim servo connector"
- note added: "BLDC PWM connector"
- note added: "Battery connection pads"
- note added: "Battery to driver logic 5V"
- note added: "Debug connector"
- note added: "Hold servo connector"
- note added: "Motor 1 connector"
- note added: "Motor 2 connector"
- note added: "Motor 3 connector"
- note added: "USB 5V to CPU logic 3v3"
- note added: "USB Power LED"
- note added: "USB port"
