File: electronics/Connectors.sch (KiCad schematic (older format))
At the start: 28 parts

Commit message: Updated titles
Other:
- note added: "1.0"
- note added: "21/10/2021"
- note added: "Connectors and voltage regulators\n"

Commit message: Made things prettier, lowered logic 3v3 LDO back to 300mA
Parts:
- removed C?: 33uF, symbol Device:C
- removed C?: 10uF, symbol Device:C
- removed U?: LM3940IT-3.3, TO254P1054X470X1955-3, symbol LM3940IT-3.3:LM3940IT-3.3
- added C?: 1uF, symbol Device:C
- added U?: NCP164, symbol Electronics:NCP164
- C?: value 0.47uF -> 1uF
Connections:
- wire segments 49 -> 46
Other:
- moved on the sheet: C?

Commit message: Updated symbols
Parts:
- R?: value 30Ohm -> 30
- R?: value 10KOhm -> 10k
- R?: value 52.3KOhm -> 52.3k
- R?: value 3.3KOhm -> 3.3k
Changed lines of the file:
@@
 AR Path="/617B7795/61AB1FFD" Ref="R?"  Part="1"
 F 0 "R?" V 6350 2400 50  0000 C CNN
-F 1 "30Ohm" V 6450 2400 50  0000 C CNN
+F 1 "30" V 6450 2400 50  0000 C CNN
 F 2 "" V 6530 2400 50  0001 C CNN
 F 3 "~" H 6600 2400 50  0001 C CNN
@@
 AR Path="/617B7795/61AB2035" Ref="R?"  Part="1"
 F 0 "R?" H 7120 3104 50  0000 L CNN
-F 1 "10KOhm" H 7120 3195 50  0000 L CNN
+F 1 "10k" H 7120 3195 50  0000 L CNN
 F 2 "" V 6980 3150 50  0001 C CNN
 F 3 "~" H 7050 3150 50  0001 C CNN
@@
 AR Path="/617B7795/61AB203B" Ref="R?"  Part="1"
 F 0 "R?" H 6981 2896 50  0000 R CNN
-F 1 "52.3KOhm" H 6981 2805 50  0000 R CNN
+F 1 "52.3k" H 6981 2805 50  0000 R CNN
 F 2 "" V 6980 2850 50  0001 C CNN
 F 3 "~" H 7050 2850 50  0001 C CNN
@@
 AR Path="/617B7795/61BC9487" Ref="R?"  Part="1"
 F 0 "R?" V 9700 4050 50  0000 C CNN
-F 1 "3.3KOhm" V 9800 4050 50  0000 C CNN
+F 1 "3.3k" V 9800 4050 50  0000 C CNN
 F 2 "" V 9880 4050 50  0001 C CNN
 F 3 "~" H 9950 4050 50  0001 C CNN

Commit message: Added reverse polarity protection
Parts:
- added Q?: BUK6Y10-30P, Package_TO_SOT_SMD:LFPAK56, symbol Electronics:BUK7M10-40EX
- J?: footprint (none) -> Electronics:3mm_pad
Connections:
- wire segments 46 -> 47
Other:
- note added: "Battery connection pads with reverse polarity protection"
- note removed: "Battery connection pads"
- moved on the sheet: C?
Changed lines of the file:
@@
 F 0 "J?" H 9779 5518 50  0000 L CNN
 F 1 "3mm_pad" H 9779 5427 50  0000 L CNN
-F 2 "" H 9950 5400 50  0001 C CNN
+F 2 "Electronics:3mm_pad" H 9950 5400 50  0001 C CNN
 F 3 "" H 9950 5400 50  0001 C CNN
 	1    9650 5350
@@
 $EndComp
 $Comp
-L Device:CP C?
-U 1 1 61AA575E
-P 9650 5050
-AR Path="/615F51F3/61AA575E" Ref="C?"  Part="1"
-AR Path="/617B7795/61AA575E" Ref="C?"  Part="1"
-F 0 "C?" H 9768 5096 50  0000 L CNN
-F 1 "4.7uF" H 9768 5005 50  0000 L CNN
-F 2 "" H 9688 4900 50  0001 C CNN
-F 3 "~" H 9650 5050 50  0001 C CNN
-	1    9650 5050
-	1    0    0    -1
-$EndComp
-$Comp
 L power:Vdrive #PWR?
 U 1 1 61AA5764
-P 9650 4800
+P 8950 4850
 AR Path="/615F51F3/61AA5764" Ref="#PWR?"  Part="1"
 AR Path="/617B7795/61AA5764" Ref="#PWR?"  Part="1"
-F 0 "#PWR?" H 9450 4650 50  0001 C CNN
-F 1 "Vdrive" H 9665 4973 50  0000 C CNN
-F 2 "" H 9650 4800 50  0001 C CNN
-F 3 "" H 9650 4800 50  0001 C CNN
-	1    9650 4800
+F 0 "#PWR?" H 8750 4700 50  0001 C CNN
+F 1 "Vdrive" H 8965 5023 50  0000 C CNN
+F 2 "" H 8950 4850 50  0001 C CNN
+F 3 "" H 8950 4850 50  0001 C CNN
+	1    8950 4850
 	1    0    0    -1
 $EndComp
-Text Notes 9200 5500 0    50   ~ 0
-Battery connection pads
+Text Notes 8400 5550 0    50   ~ 0
+Battery connection pads with reverse polarity protection
 Text Notes 9500 3550 0    50   ~ 0
 USB port
@@
 L power:Earth #PWR?
 U 1 1 61AA576C
-P 9650 5300
+P 9450 5250
 AR Path="/615F51F3/61AA576C" Ref="#PWR?"  Part="1"
 AR Path="/617B7795/61AA576C" Ref="#PWR?"  Part="1"
-F 0 "#PWR?" H 9650 5050 50  0001 C CNN
-F 1 "Earth" H 9650 5150 50  0001 C CNN
-F 2 "" H 9650 5300 50  0001 C CNN
-F 3 "~" H 9650 5300 50  0001 C CNN
-	1    9650 5300
+F 0 "#PWR?" H 9450 5000 50  0001 C CNN
+F 1 "Earth" H 9450 5100 50  0001 C CNN
+F 2 "" H 9450 5250 50  0001 C CNN
+F 3 "~" H 9450 5250 50  0001 C CNN
+	1    9450 5250
 	1    0    0    -1
 $EndComp
-Wire Wire Line
-	9650 5300 9650 5250
-Connection ~ 9650 5250
-Wire Wire Line
-	9650 5250 9650 5200
-Wire Wire Line
-	9650 4900 9650 4850
-Connection ~ 9650 4850
-Wire Wire Line
-	9650 4850 9650 4800
 $Comp
 L power:GND #PWR?
@@
 	6250 1000 6500 1000
 Connection ~ 6500 1000
+$Comp
+L Electronics:BUK7M10-40EX Q?
+U 1 1 61751376
+P 9450 4950
+F 0 "Q?" V 9792 4950 50  0000 C CNN
+F 1 "BUK6Y10-30P" V 9701 4950 50  0000 C CNN
+F 2 "Package_TO_SOT_SMD:LFPAK56" H 9650 4875 50  0001 L CIN
+F 3 "https://assets.nexperia.com/documents/data-sheet/BUK6Y10-30P.pdf" V 9450 4950 50  0001 L CNN
+	1    9450 4950
+	0    -1   -1   0
+$EndComp
+$Comp
+L Device:CP C?
+U 1 1 61AA575E
+P 8950 5000
+AR Path="/615F51F3/61AA575E" Ref="C?"  Part="1"
+AR Path="/617B7795/61AA575E" Ref="C?"  Part="1"
+F 0 "C?" H 9068 5046 50  0000 L CNN
+F 1 "4.7uF" H 9068 4955 50  0000 L CNN
+F 2 "" H 8988 4850 50  0001 C CNN
+F 3 "~" H 8950 5000 50  0001 C CNN
+	1    8950 5000
+	1    0    0    -1
+$EndComp
+Wire Wire Line
+	9450 5150 9450 5250
+Wire Wire Line
+	9650 5250 9450 5250
+Connection ~ 9450 5250
+Wire Wire Line
+	8950 5150 8950 5250
+Wire Wire Line
+	8950 5250 9450 5250
+Wire Wire Line
+	8950 4850 9250 4850
+Connection ~ 8950 4850
 $EndSCHEMATC

Commit message: Various fixes, added ESD protection
Parts:
- added U?: CM1223-02SO, symbol Electronics:CM1223-02SO
- C? (x2): value 0.1uF -> 22uF
- Q?: symbol Electronics:BUK7M10-40EX -> Transistor_FET:DMP3013SFV
Connections:
- wire segments 47 -> 48
Other:
- note added: "USB ESD protection"
- moved on the sheet: C?
Changed lines of the file:
@@
 	1    0    0    -1
 $EndComp
-Text HLabel 2750 2200 2    50   Output ~ 0
-MCU-mot2-enc_1
 Text HLabel 1950 2200 0    50   Output ~ 0
+MCU-mot2-enc_1
+Text HLabel 2750 2200 2    50   Output ~ 0
 MCU-mot2-enc_2
 $Comp
-L power:GND #PWR?
-U 1 1 618785A7
-P 2900 2050
-F 0 "#PWR?" H 2900 1800 50  0001 C CNN
-F 1 "GND" H 2988 2013 50  0000 L CNN
-F 2 "" H 2900 2050 50  0001 C CNN
-F 3 "" H 2900 2050 50  0001 C CNN
-	1    2900 2050
-	1    0    0    -1
-$EndComp
-$Comp
 L power:+3V3 #PWR?
 U 1 1 61878E48
-P 1950 2100
-F 0 "#PWR?" H 1950 1950 50  0001 C CNN
-F 1 "+3V3" H 1965 2273 50  0000 C CNN
-F 2 "" H 1950 2100 50  0001 C CNN
-F 3 "" H 1950 2100 50  0001 C CNN
-	1    1950 2100
+P 2750 2100
+F 0 "#PWR?" H 2750 1950 50  0001 C CNN
+F 1 "+3V3" H 2765 2273 50  0000 C CNN
+F 2 "" H 2750 2100 50  0001 C CNN
+F 3 "" H 2750 2100 50  0001 C CNN
+	1    2750 2100
 	1    0    0    -1
 $EndComp
-Wire Wire Line
-	2750 2100 2750 2050
-Wire Wire Line
-	2750 2050 2900 2050
 $Comp
 L 215079-4:215079-4 J?
@@
 Text Notes 2000 1600 0    50   ~ 0
 Motor 1 connector
-Text HLabel 2750 1300 2    50   Output ~ 0
-MCU-mot1-enc_1
 Text HLabel 1950 1300 0    50   Output ~ 0
+MCU-mot1-enc_1
+Text HLabel 2750 1300 2    50   Output ~ 0
 MCU-mot1-enc_2
 $Comp
 L power:GND #PWR?
 U 1 1 6187AF3C
-P 2900 1150
-F 0 "#PWR?" H 2900 900 50  0001 C CNN
-F 1 "GND" H 2988 1113 50  0000 L CNN
-F 2 "" H 2900 1150 50  0001 C CNN
-F 3 "" H 2900 1150 50  0001 C CNN
-	1    2900 1150
+P 1850 1150
+F 0 "#PWR?" H 1850 900 50  0001 C CNN
+F 1 "GND" H 1772 1113 50  0000 R CNN
+F 2 "" H 1850 1150 50  0001 C CNN
+F 3 "" H 1850 1150 50  0001 C CNN
+	1    1850 1150
 	1    0    0    -1
 $EndComp
@@
 L power:+3V3 #PWR?
 U 1 1 6187AF42
-P 1950 1200
-F 0 "#PWR?" H 1950 1050 50  0001 C CNN
-F 1 "+3V3" H 1965 1373 50  0000 C CNN
-F 2 "" H 1950 1200 50  0001 C CNN
-F 3 "" H 1950 1200 50  0001 C CNN
-	1    1950 1200
+P 2750 1200
+F 0 "#PWR?" H 2750 1050 50  0001 C CNN
+F 1 "+3V3" H 2765 1373 50  0000 C CNN
+F 2 "" H 2750 1200 50  0001 C CNN
+F 3 "" H 2750 1200 50  0001 C CNN
+	1    2750 1200
 	1    0    0    -1
 $EndComp
-Wire Wire Line
-	2750 1200 2750 1150
-Wire Wire Line
-	2750 1150 2900 1150
 $Comp
 L 215079-4:215079-4 J?
@@
 Text Notes 2000 3400 0    50   ~ 0
 Motor 3 connector
-Text HLabel 2750 3100 2    50   Output ~ 0
-MCU-mot3-enc_1
 Text HLabel 1950 3100 0    50   Output ~ 0
+MCU-mot3-enc_1
+Text HLabel 2750 3100 2    50   Output ~ 0
 MCU-mot3-enc_2
 $Comp
 L power:GND #PWR?
 U 1 1 6187B54B
-P 2900 2950
-F 0 "#PWR?" H 2900 2700 50  0001 C CNN
-F 1 "GND" H 2988 2913 50  0000 L CNN
-F 2 "" H 2900 2950 50  0001 C CNN
-F 3 "" H 2900 2950 50  0001 C CNN
-	1    2900 2950
+P 1850 2950
+F 0 "#PWR?" H 1850 2700 50  0001 C CNN
+F 1 "GND" H 1772 2913 50  0000 R CNN
+F 2 "" H 1850 2950 50  0001 C CNN
+F 3 "" H 1850 2950 50  0001 C CNN
+	1    1850 2950
 	1    0    0    -1
 $EndComp
@@
 L power:+3V3 #PWR?
 U 1 1 6187B551
-P 1950 3000
-F 0 "#PWR?" H 1950 2850 50  0001 C CNN
-F 1 "+3V3" H 1965 3173 50  0000 C CNN
-F 2 "" H 1950 3000 50  0001 C CNN
-F 3 "" H 1950 3000 50  0001 C CNN
-	1    1950 3000
+P 2750 3000
+F 0 "#PWR?" H 2750 2850 50  0001 C CNN
+F 1 "+3V3" H 2765 3173 50  0000 C CNN
+F 2 "" H 2750 3000 50  0001 C CNN
+F 3 "" H 2750 3000 50  0001 C CNN
+	1    2750 3000
 	1    0    0    -1
 $EndComp
-Wire Wire Line
-	2750 3000 2750 2950
-Wire Wire Line
-	2750 2950 2900 2950
 Text Notes 2000 2500 0    50   ~ 0
 Motor 2 connector
@@
 L Electronics:3mm_pad J?
 U 1 1 61AA5752
-P 9650 4950
+P 6300 4300
 AR Path="/615F51F3/61AA5752" Ref="J?"  Part="1"
 AR Path="/617B7795/61AA5752" Ref="J?"  Part="1"
-F 0 "J?" H 9779 5118 50  0000 L CNN
-F 1 "3mm_pad" H 9779 5027 50  0000 L CNN
-F 2 "" H 9950 5000 50  0001 C CNN
-F 3 "" H 9950 5000 50  0001 C CNN
-	1    9650 4950
+F 0 "J?" H 6429 4468 50  0000 L CNN
+F 1 "3mm_pad" H 6429 4377 50  0000 L CNN
+F 2 "" H 6600 4350 50  0001 C CNN
+F 3 "" H 6600 4350 50  0001 C CNN
+	1    6300 4300
 	1    0    0    -1
 $EndComp
@@
 L Electronics:3mm_pad J?
 U 1 1 61AA5758
-P 9650 5350
+P 6300 4700
 AR Path="/615F51F3/61AA5758" Ref="J?"  Part="1"
 AR Path="/617B7795/61AA5758" Ref="J?"  Part="1"
-F 0 "J?" H 9779 5518 50  0000 L CNN
-F 1 "3mm_pad" H 9779 5427 50  0000 L CNN
-F 2 "Electronics:3mm_pad" H 9950 5400 50  0001 C CNN
-F 3 "" H 9950 5400 50  0001 C CNN
-	1    9650 5350
+F 0 "J?" H 6429 4868 50  0000 L CNN
+F 1 "3mm_pad" H 6429 4777 50  0000 L CNN
+F 2 "Electronics:3mm_pad" H 6600 4750 50  0001 C CNN
+F 3 "" H 6600 4750 50  0001 C CNN
+	1    6300 4700
 	1    0    0    -1
 $EndComp
@@
 L power:Vdrive #PWR?
 U 1 1 61AA5764
-P 8950 4850
+P 5600 4200
 AR Path="/615F51F3/61AA5764" Ref="#PWR?"  Part="1"
 AR Path="/617B7795/61AA5764" Ref="#PWR?"  Part="1"
-F 0 "#PWR?" H 8750 4700 50  0001 C CNN
-F 1 "Vdrive" H 8965 5023 50  0000 C CNN
-F 2 "" H 8950 4850 50  0001 C CNN
-F 3 "" H 8950 4850 50  0001 C CNN
-	1    8950 4850
+F 0 "#PWR?" H 5400 4050 50  0001 C CNN
+F 1 "Vdrive" H 5615 4373 50  0000 C CNN
+F 2 "" H 5600 4200 50  0001 C CNN
+F 3 "" H 5600 4200 50  0001 C CNN
+	1    5600 4200
 	1    0    0    -1
 $EndComp
-Text Notes 8400 5550 0    50   ~ 0
+Text Notes 5050 4900 0    50   ~ 0
 Battery connection pads with reverse polarity protection
 Text Notes 9500 3550 0    50   ~ 0
@@
 L power:Earth #PWR?
 U 1 1 61AA576C
-P 9450 5250
+P 6100 4600
 AR Path="/615F51F3/61AA576C" Ref="#PWR?"  Part="1"
 AR Path="/617B7795/61AA576C" Ref="#PWR?"  Part="1"
-F 0 "#PWR?" H 9450 5000 50  0001 C CNN
-F 1 "Earth" H 9450 5100 50  0001 C CNN
-F 2 "" H 9450 5250 50  0001 C CNN
-F 3 "~" H 9450 5250 50  0001 C CNN
-	1    9450 5250
+F 0 "#PWR?" H 6100 4350 50  0001 C CNN
+F 1 "Earth" H 6100 4450 50  0001 C CNN
+F 2 "" H 6100 4600 50  0001 C CNN
+F 3 "~" H 6100 4600 50  0001 C CNN
+	1    6100 4600
 	1    0    0    -1
 $EndComp
@@
 AR Path="/617B7795/61AB204A" Ref="C?"  Part="1"
 F 0 "C?" H 7465 2896 50  0000 L CNN
-F 1 "0.1uF" H 7465 2805 50  0000 L CNN
+F 1 "22uF" H 7465 2805 50  0000 L CNN
 F 2 "" H 7388 2700 50  0001 C CNN
 F 3 "~" H 7350 2850 50  0001 C CNN
@@
 AR Path="/617B7795/61AB2050" Ref="C?"  Part="1"
 F 0 "C?" H 7915 2896 50  0000 L CNN
-F 1 "0.1uF" H 7915 2805 50  0000 L CNN
+F 1 "22uF" H 7915 2805 50  0000 L CNN
 F 2 "" H 7838 2700 50  0001 C CNN
 F 3 "~" H 7800 2850 50  0001 C CNN
@@
 Connection ~ 6500 1000
 $Comp
-L Electronics:BUK7M10-40EX Q?
+L Transistor_FET:DMP3013SFV Q?
 U 1 1 61751376
-P 9450 4950
-F 0 "Q?" V 9792 4950 50  0000 C CNN
-F 1 "BUK6Y10-30P" V 9701 4950 50  0000 C CNN
-F 2 "Package_TO_SOT_SMD:LFPAK56" H 9650 4875 50  0001 L CIN
-F 3 "https://assets.nexperia.com/documents/data-sheet/BUK6Y10-30P.pdf" V 9450 4950 50  0001 L CNN
-	1    9450 4950
+P 6100 4300
+F 0 "Q?" V 6442 4300 50  0000 C CNN
+F 1 "BUK6Y10-30P" V 6351 4300 50  0000 C CNN
+F 2 "Package_TO_SOT_SMD:LFPAK56" H 6300 4225 50  0001 L CIN
+F 3 "https://assets.nexperia.com/documents/data-sheet/BUK6Y10-30P.pdf" V 6100 4300 50  0001 L CNN
+	1    6100 4300
 	0    -1   -1   0
 $EndComp
@@
 L Device:CP C?
 U 1 1 61AA575E
-P 8950 5000
+P 5600 4350
 AR Path="/615F51F3/61AA575E" Ref="C?"  Part="1"
 AR Path="/617B7795/61AA575E" Ref="C?"  Part="1"
-F 0 "C?" H 9068 5046 50  0000 L CNN
-F 1 "4.7uF" H 9068 4955 50  0000 L CNN
-F 2 "" H 8988 4850 50  0001 C CNN
-F 3 "~" H 8950 5000 50  0001 C CNN
-	1    8950 5000
+F 0 "C?" H 5718 4396 50  0000 L CNN
+F 1 "4.7uF" H 5718 4305 50  0000 L CNN
+F 2 "" H 5638 4200 50  0001 C CNN
+F 3 "~" H 5600 4350 50  0001 C CNN
+	1    5600 4350
+	1    0    0    -1
+$EndComp
+Wire Wire Line
+	6100 4500 6100 4600
+Wire Wire Line
+	6300 4600 6100 4600
+Connection ~ 6100 4600
+Wire Wire Line
+	5600 4500 5600 4600
+Wire Wire Line
+	5600 4600 6100 4600
+Wire Wire Line
+	5600 4200 5900 4200
+Connection ~ 5600 4200
+Wire Wire Line
+	1850 1150 1950 1150
+Wire Wire Line
+	1950 1150 1950 1200
+$Comp
+L power:GND #PWR?
+U 1 1 618785A7
+P 1850 2050
+F 0 "#PWR?" H 1850 1800 50  0001 C CNN
+F 1 "GND" H 1772 2013 50  0000 R CNN
+F 2 "" H 1850 2050 50  0001 C CNN
+F 3 "" H 1850 2050 50  0001 C CNN
+	1    1850 2050
 	1    0    0    -1
 $EndComp
 Wire Wire Line
-	9450 5150 9450 5250
+	1850 2050 1950 2050
 Wire Wire Line
-	9650 5250 9450 5250
-Connection ~ 9450 5250
+	1950 2050 1950 2100
 Wire Wire Line
-	8950 5150 8950 5250
+	1850 2950 1950 2950
 Wire Wire Line
-	8950 5250 9450 5250
+	1950 2950 1950 3000
+$Comp
+L Electronics:CM1223-02SO U?
+U 1 1 617C765D
+P 9700 5000
+F 0 "U?" H 9750 5575 50  0000 C CNN
+F 1 "CM1223-02SO" H 9750 5484 50  0000 C CNN
+F 2 "" H 9750 4950 50  0001 C CNN
+F 3 "" H 9750 4950 50  0001 C CNN
+	1    9700 5000
+	1    0    0    -1
+$EndComp
+Text HLabel 9450 4850 0    50   BiDi ~ 0
+MCU-USB_DP
+Text HLabel 9450 4750 0    50   BiDi ~ 0
+MCU-USB_DM
+$Comp
+L power:+5VL #PWR?
+U 1 1 617D79CC
+P 9350 4650
+AR Path="/615F51F3/617D79CC" Ref="#PWR?"  Part="1"
+AR Path="/617B7795/617D79CC" Ref="#PWR?"  Part="1"
+F 0 "#PWR?" H 9350 4500 50  0001 C CNN
+F 1 "+5VL" H 9365 4823 50  0000 C CNN
+F 2 "" H 9350 4650 50  0001 C CNN
+F 3 "" H 9350 4650 50  0001 C CNN
+	1    9350 4650
+	1    0    0    -1
+$EndComp
+$Comp
+L power:GND #PWR?
+U 1 1 617DD220
+P 10050 4800
+AR Path="/615F51F3/617DD220" Ref="#PWR?"  Part="1"
+AR Path="/617B7795/617DD220" Ref="#PWR?"  Part="1"
+F 0 "#PWR?" H 10050 4550 50  0001 C CNN
+F 1 "GND" H 10055 4627 50  0000 C CNN
+F 2 "" H 10050 4800 50  0001 C CNN
+F 3 "" H 10050 4800 50  0001 C CNN
+	1    10050 4800
+	1    0    0    -1
+$EndComp
 Wire Wire Line
-	8950 4850 9250 4850
-Connection ~ 8950 4850
+	9350 4650 9450 4650
+Text Notes 9200 5250 0    50   ~ 0
+USB ESD protection
 $EndSCHEMATC

Commit message: Updated rev numbers
Other:
- note added: "1.1"
- note added: "24/10/2021"
- note removed: "1.0"
- note removed: "21/10/2021"
Changed lines of the file:
@@
 Connectors and voltage regulators\n
 Text Notes 8100 7650 0    50   ~ 0
-21/10/2021
+24/10/2021
 Text Notes 10550 7650 0    50   ~ 0
-1.0
+1.1
 $Comp
 L Device:C C?

Commit message: Replaced 5V regulator
Parts:
- removed C?: 0.1uF, symbol Device:C
- removed C?: 10uF, symbol Device:C
- removed C? (x2): 22uF, symbol Device:C
- removed R?: 10k, symbol Device:R
- removed R?: 52.3k, symbol Device:R
- removed U?: TPS56339DDC, Package_TO_SOT_SMD:SOT-23-6, symbol Regulator_Switching:TPS56339DDC
- added ?: LM20323MH_NOPB, MXA20A, symbol LM20323MH_NOPB:LM20323MH_NOPB
- added C? (x2): 0.1uF, symbol Device:C
- added C? (x3): 47uF, symbol Device:CP
- added C? (x2): 6.8nF, symbol Device:C
- added C?: 10uF, symbol Device:C
- added C?: 10pF, symbol Device:C
- added R?: 10k, symbol Device:R
- added R?: 47k, symbol Device:R
- added R?: 7.5k, symbol Device:R
- L?: value 5.6uH -> 10uH
- R?: value 30 -> 56k
Connections:
- wire segments 48 -> 67
Other:
- moved on the sheet: C?

Commit message: MOSFET fix
Connections:
- wire segments 67 -> 64
Other:
- moved on the sheet: C?
Changed lines of the file:
@@
 L Electronics:3mm_pad J?
 U 1 1 61AA5752
-P 6300 4300
+P 5800 4450
 AR Path="/615F51F3/61AA5752" Ref="J?"  Part="1"
 AR Path="/617B7795/61AA5752" Ref="J?"  Part="1"
-F 0 "J?" H 6429 4468 50  0000 L CNN
-F 1 "3mm_pad" H 6429 4377 50  0000 L CNN
-F 2 "" H 6600 4350 50  0001 C CNN
-F 3 "" H 6600 4350 50  0001 C CNN
-	1    6300 4300
-	1    0    0    -1
+F 0 "J?" H 5929 4618 50  0000 L CNN
+F 1 "3mm_pad" H 5929 4527 50  0000 L CNN
+F 2 "" H 6100 4500 50  0001 C CNN
+F 3 "" H 6100 4500 50  0001 C CNN
+	1    5800 4450
+	-1   0    0    1
 $EndComp
 $Comp
 L Electronics:3mm_pad J?
 U 1 1 61AA5758
-P 6300 4700
+P 5800 4150
 AR Path="/615F51F3/61AA5758" Ref="J?"  Part="1"
 AR Path="/617B7795/61AA5758" Ref="J?"  Part="1"
-F 0 "J?" H 6429 4868 50  0000 L CNN
-F 1 "3mm_pad" H 6429 4777 50  0000 L CNN
-F 2 "Electronics:3mm_pad" H 6600 4750 50  0001 C CNN
-F 3 "" H 6600 4750 50  0001 C CNN
-	1    6300 4700
-	1    0    0    -1
+F 0 "J?" H 5929 4318 50  0000 L CNN
+F 1 "3mm_pad" H 5929 4227 50  0000 L CNN
+F 2 "Electronics:3mm_pad" H 6100 4200 50  0001 C CNN
+F 3 "" H 6100 4200 50  0001 C CNN
+	1    5800 4150
+	-1   0    0    1
 $EndComp
 $Comp
 L power:Vdrive #PWR?
 U 1 1 61AA5764
-P 5600 4200
+P 6550 4250
 AR Path="/615F51F3/61AA5764" Ref="#PWR?"  Part="1"
 AR Path="/617B7795/61AA5764" Ref="#PWR?"  Part="1"
-F 0 "#PWR?" H 5400 4050 50  0001 C CNN
-F 1 "Vdrive" H 5615 4373 50  0000 C CNN
-F 2 "" H 5600 4200 50  0001 C CNN
-F 3 "" H 5600 4200 50  0001 C CNN
-	1    5600 4200
+F 0 "#PWR?" H 6350 4100 50  0001 C CNN
+F 1 "Vdrive" H 6565 4423 50  0000 C CNN
+F 2 "" H 6550 4250 50  0001 C CNN
+F 3 "" H 6550 4250 50  0001 C CNN
+	1    6550 4250
 	1    0    0    -1
 $EndComp
@@
 L power:Earth #PWR?
 U 1 1 61AA576C
-P 6100 4600
+P 6000 4550
 AR Path="/615F51F3/61AA576C" Ref="#PWR?"  Part="1"
 AR Path="/617B7795/61AA576C" Ref="#PWR?"  Part="1"
-F 0 "#PWR?" H 6100 4350 50  0001 C CNN
-F 1 "Earth" H 6100 4450 50  0001 C CNN
-F 2 "" H 6100 4600 50  0001 C CNN
-F 3 "~" H 6100 4600 50  0001 C CNN
-	1    6100 4600
+F 0 "#PWR?" H 6000 4300 50  0001 C CNN
+F 1 "Earth" H 6000 4400 50  0001 C CNN
+F 2 "" H 6000 4550 50  0001 C CNN
+F 3 "~" H 6000 4550 50  0001 C CNN
+	1    6000 4550
 	1    0    0    -1
 $EndComp
@@
 L Transistor_FET:DMP3013SFV Q?
 U 1 1 61751376
-P 6100 4300
-F 0 "Q?" V 6442 4300 50  0000 C CNN
-F 1 "BUK6Y10-30P" V 6351 4300 50  0000 C CNN
-F 2 "Package_TO_SOT_SMD:LFPAK56" H 6300 4225 50  0001 L CIN
-F 3 "https://assets.nexperia.com/documents/data-sheet/BUK6Y10-30P.pdf" V 6100 4300 50  0001 L CNN
-	1    6100 4300
+P 6000 4350
+F 0 "Q?" V 6342 4350 50  0000 C CNN
+F 1 "BUK6Y10-30P" V 6251 4350 50  0000 C CNN
+F 2 "Package_TO_SOT_SMD:LFPAK56" H 6200 4275 50  0001 L CIN
+F 3 "https://assets.nexperia.com/documents/data-sheet/BUK6Y10-30P.pdf" V 6000 4350 50  0001 L CNN
+	1    6000 4350
 	0    -1   -1   0
 $EndComp
@@
 L Device:CP C?
 U 1 1 61AA575E
-P 5600 4350
+P 6550 4400
 AR Path="/615F51F3/61AA575E" Ref="C?"  Part="1"
 AR Path="/617B7795/61AA575E" Ref="C?"  Part="1"
-F 0 "C?" H 5718 4396 50  0000 L CNN
-F 1 "4.7uF" H 5718 4305 50  0000 L CNN
-F 2 "" H 5638 4200 50  0001 C CNN
-F 3 "~" H 5600 4350 50  0001 C CNN
-	1    5600 4350
+F 0 "C?" H 6668 4446 50  0000 L CNN
+F 1 "4.7uF" H 6668 4355 50  0000 L CNN
+F 2 "" H 6588 4250 50  0001 C CNN
+F 3 "~" H 6550 4400 50  0001 C CNN
+	1    6550 4400
 	1    0    0    -1
 $EndComp
 Wire Wire Line
-	6100 4500 6100 4600
-Wire Wire Line
-	6300 4600 6100 4600
-Connection ~ 6100 4600
-Wire Wire Line
-	5600 4500 5600 4600
-Wire Wire Line
-	5600 4600 6100 4600
-Wire Wire Line
-	5600 4200 5900 4200
-Connection ~ 5600 4200
-Wire Wire Line
 	1850 1150 1950 1150
 Wire Wire Line
@@
 	1    0    0    -1
 $EndComp
+Wire Wire Line
+	5800 4550 6000 4550
+Connection ~ 6000 4550
+Wire Wire Line
+	6200 4250 6550 4250
+Connection ~ 6550 4250
+$Comp
+L power:Earth #PWR?
+U 1 1 61794771
+P 6550 4550
+AR Path="/615F51F3/61794771" Ref="#PWR?"  Part="1"
+AR Path="/617B7795/61794771" Ref="#PWR?"  Part="1"
+F 0 "#PWR?" H 6550 4300 50  0001 C CNN
+F 1 "Earth" H 6550 4400 50  0001 C CNN
+F 2 "" H 6550 4550 50  0001 C CNN
+F 3 "~" H 6550 4550 50  0001 C CNN
+	1    6550 4550
+	1    0    0    -1
+$EndComp
