File: electronics/Driver.sch (KiCad schematic (older format))
At the start: 21 parts

Commit message: Added isolators, updated CPU pins
Parts:
- added J? (x6): 3mm_pad, symbol Electronics:3mm_pad
Connections:
- net labels added: Earth, MOT_off, MOT_sleep
- net labels removed: MOT1out_1, MOT1out_2, MOT2out_1, MOT2out_2, MOT3out_1, MOT3out_2, MOTSleep, MOToff

Commit message: Added connectors, started relabeling pins
Changed lines of the file:
@@
 $Descr A4 11693 8268
 encoding utf-8
-Sheet 3 4
+Sheet 3 5
 Title ""
 Date ""
@@
 	2800 1500 2800 1600
 $Comp
-L power:GND #PWR?
+L power:GND #PWR0125
 U 1 1 6160C826
 P 2800 1600
-F 0 "#PWR?" H 2800 1350 50  0001 C CNN
+F 0 "#PWR0125" H 2800 1350 50  0001 C CNN
 F 1 "GND" H 2805 1427 50  0000 C CNN
 F 2 "" H 2800 1600 50  0001 C CNN
@@
 $EndComp
 $Comp
-L power:Vdrive #PWR?
+L power:Vdrive #PWR0126
 U 1 1 6160C82C
 P 2300 1050
-F 0 "#PWR?" H 2100 900 50  0001 C CNN
+F 0 "#PWR0126" H 2100 900 50  0001 C CNN
 F 1 "Vdrive" H 2315 1223 50  0000 C CNN
 F 2 "" H 2300 1050 50  0001 C CNN
@@
 	6450 1500 6450 1600
 $Comp
-L power:GND #PWR?
+L power:GND #PWR0127
 U 1 1 6160C89D
 P 6450 1600
-F 0 "#PWR?" H 6450 1350 50  0001 C CNN
+F 0 "#PWR0127" H 6450 1350 50  0001 C CNN
 F 1 "GND" H 6455 1427 50  0000 C CNN
 F 2 "" H 6450 1600 50  0001 C CNN
@@
 $EndComp
 $Comp
-L power:Vdrive #PWR?
+L power:Vdrive #PWR0128
 U 1 1 6160C8A3
 P 5950 1050
-F 0 "#PWR?" H 5750 900 50  0001 C CNN
+F 0 "#PWR0128" H 5750 900 50  0001 C CNN
 F 1 "Vdrive" H 5965 1223 50  0000 C CNN
 F 2 "" H 5950 1050 50  0001 C CNN
@@
 	9900 1500 9900 1600
 $Comp
-L power:GND #PWR?
+L power:GND #PWR0129
 U 1 1 6160C914
 P 9900 1600
-F 0 "#PWR?" H 9900 1350 50  0001 C CNN
+F 0 "#PWR0129" H 9900 1350 50  0001 C CNN
 F 1 "GND" H 9905 1427 50  0000 C CNN
 F 2 "" H 9900 1600 50  0001 C CNN
@@
 $EndComp
 $Comp
-L power:Vdrive #PWR?
+L power:Vdrive #PWR0130
 U 1 1 6160C91A
 P 9400 1050
-F 0 "#PWR?" H 9200 900 50  0001 C CNN
+F 0 "#PWR0130" H 9200 900 50  0001 C CNN
 F 1 "Vdrive" H 9415 1223 50  0000 C CNN
 F 2 "" H 9400 1050 50  0001 C CNN
@@
 Text Label 8500 1900 0    50   ~ 0
 MOT3en_2
-Text Label 8500 1800 0    50   ~ 0
-MOT3en_1
 $Comp
 L Device:R_US R?
@@
 	8500 1900 8950 1900
 $Comp
-L power:Earth #PWR?
+L power:Earth #PWR0131
 U 1 1 616D1C7A
 P 9850 3050
-F 0 "#PWR?" H 9850 2800 50  0001 C CNN
+F 0 "#PWR0131" H 9850 2800 50  0001 C CNN
 F 1 "Earth" H 9850 2900 50  0001 C CNN
 F 2 "" H 9850 3050 50  0001 C CNN
@@
 $EndComp
 $Comp
-L power:Earth #PWR?
+L power:Earth #PWR0132
 U 1 1 616EF01B
 P 9400 2950
-F 0 "#PWR?" H 9400 2700 50  0001 C CNN
+F 0 "#PWR0132" H 9400 2700 50  0001 C CNN
 F 1 "Earth" H 9400 2800 50  0001 C CNN
 F 2 "" H 9400 2950 50  0001 C CNN
@@
 $EndComp
 $Comp
-L power:Earth #PWR?
+L power:Earth #PWR0133
 U 1 1 616F0746
 P 8850 2900
-F 0 "#PWR?" H 8850 2650 50  0001 C CNN
+F 0 "#PWR0133" H 8850 2650 50  0001 C CNN
 F 1 "Earth" H 8850 2750 50  0001 C CNN
 F 2 "" H 8850 2900 50  0001 C CNN
@@
 $EndComp
 $Comp
-L power:Earth #PWR?
+L power:Earth #PWR0134
 U 1 1 616F1D4C
 P 8700 2850
-F 0 "#PWR?" H 8700 2600 50  0001 C CNN
+F 0 "#PWR0134" H 8700 2600 50  0001 C CNN
 F 1 "Earth" H 8700 2700 50  0001 C CNN
 F 2 "" H 8700 2850 50  0001 C CNN
@@
 $EndComp
 $Comp
-L power:Earth #PWR?
+L power:Earth #PWR0135
 U 1 1 616F3423
 P 8450 2750
-F 0 "#PWR?" H 8450 2500 50  0001 C CNN
+F 0 "#PWR0135" H 8450 2500 50  0001 C CNN
 F 1 "Earth" H 8450 2600 50  0001 C CNN
 F 2 "" H 8450 2750 50  0001 C CNN
@@
 $EndComp
 $Comp
-L power:Earth #PWR?
+L power:Earth #PWR0136
 U 1 1 616F565E
 P 6400 3050
-F 0 "#PWR?" H 6400 2800 50  0001 C CNN
+F 0 "#PWR0136" H 6400 2800 50  0001 C CNN
 F 1 "Earth" H 6400 2900 50  0001 C CNN
 F 2 "" H 6400 3050 50  0001 C CNN
@@
 $EndComp
 $Comp
-L power:Earth #PWR?
+L power:Earth #PWR0137
 U 1 1 616F6E00
 P 5950 2950
-F 0 "#PWR?" H 5950 2700 50  0001 C CNN
+F 0 "#PWR0137" H 5950 2700 50  0001 C CNN
 F 1 "Earth" H 5950 2800 50  0001 C CNN
 F 2 "" H 5950 2950 50  0001 C CNN
@@
 $EndComp
 $Comp
-L power:Earth #PWR?
+L power:Earth #PWR0138
 U 1 1 616F85FE
 P 5400 2900
-F 0 "#PWR?" H 5400 2650 50  0001 C CNN
+F 0 "#PWR0138" H 5400 2650 50  0001 C CNN
 F 1 "Earth" H 5400 2750 50  0001 C CNN
 F 2 "" H 5400 2900 50  0001 C CNN
@@
 $EndComp
 $Comp
-L power:Earth #PWR?
+L power:Earth #PWR0139
 U 1 1 616F9D5B
 P 5250 2850
-F 0 "#PWR?" H 5250 2600 50  0001 C CNN
+F 0 "#PWR0139" H 5250 2600 50  0001 C CNN
 F 1 "Earth" H 5250 2700 50  0001 C CNN
 F 2 "" H 5250 2850 50  0001 C CNN
@@
 $EndComp
 $Comp
-L power:Earth #PWR?
+L power:Earth #PWR0140
 U 1 1 616FB4B8
 P 5000 2750
-F 0 "#PWR?" H 5000 2500 50  0001 C CNN
+F 0 "#PWR0140" H 5000 2500 50  0001 C CNN
 F 1 "Earth" H 5000 2600 50  0001 C CNN
 F 2 "" H 5000 2750 50  0001 C CNN
@@
 $EndComp
 $Comp
-L power:Earth #PWR?
+L power:Earth #PWR0141
 U 1 1 616FD602
 P 2750 3050
-F 0 "#PWR?" H 2750 2800 50  0001 C CNN
+F 0 "#PWR0141" H 2750 2800 50  0001 C CNN
 F 1 "Earth" H 2750 2900 50  0001 C CNN
 F 2 "" H 2750 3050 50  0001 C CNN
@@
 $EndComp
 $Comp
-L power:Earth #PWR?
+L power:Earth #PWR0142
 U 1 1 616FECDD
 P 2300 2950
-F 0 "#PWR?" H 2300 2700 50  0001 C CNN
+F 0 "#PWR0142" H 2300 2700 50  0001 C CNN
 F 1 "Earth" H 2300 2800 50  0001 C CNN
 F 2 "" H 2300 2950 50  0001 C CNN
@@
 $EndComp
 $Comp
-L power:Earth #PWR?
+L power:Earth #PWR0143
 U 1 1 6170042B
 P 1750 2900
-F 0 "#PWR?" H 1750 2650 50  0001 C CNN
+F 0 "#PWR0143" H 1750 2650 50  0001 C CNN
 F 1 "Earth" H 1750 2750 50  0001 C CNN
 F 2 "" H 1750 2900 50  0001 C CNN
@@
 $EndComp
 $Comp
-L power:Earth #PWR?
+L power:Earth #PWR0144
 U 1 1 61701B1D
 P 1600 2850
-F 0 "#PWR?" H 1600 2600 50  0001 C CNN
+F 0 "#PWR0144" H 1600 2600 50  0001 C CNN
 F 1 "Earth" H 1600 2700 50  0001 C CNN
 F 2 "" H 1600 2850 50  0001 C CNN
@@
 $EndComp
 $Comp
-L power:Earth #PWR?
+L power:Earth #PWR0145
 U 1 1 61703249
 P 1350 2750
-F 0 "#PWR?" H 1350 2500 50  0001 C CNN
+F 0 "#PWR0145" H 1350 2500 50  0001 C CNN
 F 1 "Earth" H 1350 2600 50  0001 C CNN
 F 2 "" H 1350 2750 50  0001 C CNN
@@
 Text Label 1400 2000 0    50   ~ 0
 MOT_sleep
+Text HLabel 8500 1800 0    50   Input ~ 0
+MOT3en_1
 $EndSCHEMATC

Commit message: Another restructure, added CPU pins, updated V regulators
Connections:
- wire segments 69 -> 57
Other:
- note added: "Motor 1 driver"
- note added: "Motor 2 driver"
- note added: "Motor 3 driver"
Changed lines of the file:
@@
 $Descr A4 11693 8268
 encoding utf-8
-Sheet 3 5
+Sheet 2 3
 Title ""
 Date ""
@@
 Wire Wire Line
 	1750 2800 1750 2900
-Text Label 1400 1900 0    50   ~ 0
-MOT1en_2
-Text Label 1400 1800 0    50   ~ 0
-MOT1en_1
 $Comp
 L Device:R_US R?
@@
 	1    0    0    -1
 $EndComp
-Wire Wire Line
-	1400 1800 1850 1800
-Wire Wire Line
-	1400 1900 1850 1900
 $Comp
 L Device:C C?
@@
 Wire Wire Line
 	5400 2800 5400 2900
-Text Label 5050 1900 0    50   ~ 0
-MOT2en_2
-Text Label 5050 1800 0    50   ~ 0
-MOT2en_1
 $Comp
 L Device:R_US R?
@@
 	1    0    0    -1
 $EndComp
-Wire Wire Line
-	5050 1800 5500 1800
-Wire Wire Line
-	5050 1900 5500 1900
 $Comp
 L Device:C C?
@@
 Wire Wire Line
 	8850 2800 8850 2900
-Wire Wire Line
-	8500 2200 8950 2200
-Text Label 8500 2200 0    50   ~ 0
-MOT_off
-Wire Wire Line
-	8500 2000 8950 2000
-Text Label 8500 2000 0    50   ~ 0
-MOT_sleep
-Text Label 8500 1900 0    50   ~ 0
-MOT3en_2
 $Comp
 L Device:R_US R?
@@
 	1    0    0    -1
 $EndComp
-Wire Wire Line
-	8500 1800 8950 1800
-Wire Wire Line
-	8500 1900 8950 1900
 $Comp
 L power:Earth #PWR0131
@@
 Connection ~ 9950 2100
 Connection ~ 9950 2400
-Wire Wire Line
-	5050 2200 5500 2200
-Text Label 5050 2200 0    50   ~ 0
+Text HLabel 8950 1800 0    50   Input ~ 0
+MOT3en_1
+Text HLabel 8950 1900 0    50   Input ~ 0
+MOT3en_2
+Text HLabel 8950 2000 0    50   Input ~ 0
+MOT_sleep
+Text HLabel 8950 2200 0    50   Input ~ 0
 MOT_off
-Wire Wire Line
-	5050 2000 5500 2000
-Text Label 5050 2000 0    50   ~ 0
+Text HLabel 1850 1800 0    50   Input ~ 0
+MOT1en_1
+Text HLabel 1850 1900 0    50   Input ~ 0
+MOT1en_2
+Text HLabel 5500 1800 0    50   Input ~ 0
+MOT2en_1
+Text HLabel 5500 1900 0    50   Input ~ 0
+MOT2en_2
+Text HLabel 5500 2000 0    50   Input ~ 0
 MOT_sleep
-Wire Wire Line
-	1400 2200 1850 2200
-Text Label 1400 2200 0    50   ~ 0
+Text HLabel 5500 2200 0    50   Input ~ 0
 MOT_off
-Wire Wire Line
-	1400 2000 1850 2000
-Text Label 1400 2000 0    50   ~ 0
+Text HLabel 1850 2000 0    50   Input ~ 0
 MOT_sleep
-Text HLabel 8500 1800 0    50   Input ~ 0
-MOT3en_1
+Text HLabel 1850 2200 0    50   Input ~ 0
+MOT_off
+Text Notes 2050 3450 0    50   ~ 0
+Motor 1 driver
+Text Notes 5700 3500 0    50   ~ 0
+Motor 2 driver
+Text Notes 9250 3450 0    50   ~ 0
+Motor 3 driver
 $EndSCHEMATC

Commit message: Updated titles
Other:
- note added: "1.0"
- note added: "21/10/2021"
- note added: "Kurkkumopo HBridge driver"

Commit message: Updated symbols
Parts:
- removed R? (x6): 100k, Resistor_SMD:R_0603_1608Metric_Pad0.98x0.95mm_HandSolder, symbol Device:R_US
- removed R? (x3): 2.7k, Resistor_SMD:R_0603_1608Metric_Pad0.98x0.95mm_HandSolder, symbol Device:R_US
- added R? (x6): 100k, symbol Device:R
- added R? (x3): 2.7k, symbol Device:R
Changed lines of the file:
@@
 Wire Wire Line
 	1750 2800 1750 2900
-$Comp
-L Device:R_US R?
-U 1 1 6160C874
-P 1350 2600
-F 0 "R?" H 1250 2700 50  0000 C CNN
-F 1 "100k" H 1200 2600 50  0000 C CNN
-F 2 "Resistor_SMD:R_0603_1608Metric_Pad0.98x0.95mm_HandSolder" V 1390 2590 50  0001 C CNN
-F 3 "~" H 1350 2600 50  0001 C CNN
-	1    1350 2600
-	1    0    0    -1
-$EndComp
-$Comp
-L Device:R_US R?
-U 1 1 6160C87A
-P 1600 2700
-F 0 "R?" H 1500 2800 50  0000 C CNN
-F 1 "100k" H 1450 2700 50  0000 C CNN
-F 2 "Resistor_SMD:R_0603_1608Metric_Pad0.98x0.95mm_HandSolder" V 1640 2690 50  0001 C CNN
-F 3 "~" H 1600 2700 50  0001 C CNN
-	1    1600 2700
-	1    0    0    -1
-$EndComp
 Wire Wire Line
 	1600 2550 1850 2550
@@
 	1350 2450 1850 2450
 $Comp
-L Device:R_US R?
-U 1 1 6160C888
-P 2750 2900
-F 0 "R?" H 2818 2946 50  0000 L CNN
-F 1 "2.7k" H 2818 2855 50  0000 L CNN
-F 2 "Resistor_SMD:R_0603_1608Metric_Pad0.98x0.95mm_HandSolder" V 2790 2890 50  0001 C CNN
-F 3 "~" H 2750 2900 50  0001 C CNN
-	1    2750 2900
-	1    0    0    -1
-$EndComp
-$Comp
 L Device:C C?
 U 1 1 6160C896
@@
 Wire Wire Line
 	5400 2800 5400 2900
-$Comp
-L Device:R_US R?
-U 1 1 6160C8EB
-P 5000 2600
-F 0 "R?" H 4900 2700 50  0000 C CNN
-F 1 "100k" H 4850 2600 50  0000 C CNN
-F 2 "Resistor_SMD:R_0603_1608Metric_Pad0.98x0.95mm_HandSolder" V 5040 2590 50  0001 C CNN
-F 3 "~" H 5000 2600 50  0001 C CNN
-	1    5000 2600
-	1    0    0    -1
-$EndComp
-$Comp
-L Device:R_US R?
-U 1 1 6160C8F1
-P 5250 2700
-F 0 "R?" H 5150 2800 50  0000 C CNN
-F 1 "100k" H 5100 2700 50  0000 C CNN
-F 2 "Resistor_SMD:R_0603_1608Metric_Pad0.98x0.95mm_HandSolder" V 5290 2690 50  0001 C CNN
-F 3 "~" H 5250 2700 50  0001 C CNN
-	1    5250 2700
-	1    0    0    -1
-$EndComp
 Wire Wire Line
 	5250 2550 5500 2550
@@
 	5000 2450 5500 2450
 $Comp
-L Device:R_US R?
-U 1 1 6160C8FF
-P 6400 2900
-F 0 "R?" H 6468 2946 50  0000 L CNN
-F 1 "2.7k" H 6468 2855 50  0000 L CNN
-F 2 "Resistor_SMD:R_0603_1608Metric_Pad0.98x0.95mm_HandSolder" V 6440 2890 50  0001 C CNN
-F 3 "~" H 6400 2900 50  0001 C CNN
-	1    6400 2900
-	1    0    0    -1
-$EndComp
-$Comp
 L Electronics:DRV8243 U?
 U 1 1 6160C905
@@
 Wire Wire Line
 	8850 2800 8850 2900
-$Comp
-L Device:R_US R?
-U 1 1 6160C962
-P 8450 2600
-F 0 "R?" H 8350 2700 50  0000 C CNN
-F 1 "100k" H 8300 2600 50  0000 C CNN
-F 2 "Resistor_SMD:R_0603_1608Metric_Pad0.98x0.95mm_HandSolder" V 8490 2590 50  0001 C CNN
-F 3 "~" H 8450 2600 50  0001 C CNN
-	1    8450 2600
-	1    0    0    -1
-$EndComp
-$Comp
-L Device:R_US R?
-U 1 1 6160C968
-P 8700 2700
-F 0 "R?" H 8600 2800 50  0000 C CNN
-F 1 "100k" H 8550 2700 50  0000 C CNN
-F 2 "Resistor_SMD:R_0603_1608Metric_Pad0.98x0.95mm_HandSolder" V 8740 2690 50  0001 C CNN
-F 3 "~" H 8700 2700 50  0001 C CNN
-	1    8700 2700
-	1    0    0    -1
-$EndComp
 Wire Wire Line
 	8700 2550 8950 2550
@@
 	8450 2450 8950 2450
 $Comp
-L Device:R_US R?
-U 1 1 6160C976
-P 9850 2900
-F 0 "R?" H 9918 2946 50  0000 L CNN
-F 1 "2.7k" H 9918 2855 50  0000 L CNN
-F 2 "Resistor_SMD:R_0603_1608Metric_Pad0.98x0.95mm_HandSolder" V 9890 2890 50  0001 C CNN
-F 3 "~" H 9850 2900 50  0001 C CNN
-	1    9850 2900
-	1    0    0    -1
-$EndComp
-$Comp
 L power:Earth #PWR0131
 U 1 1 616D1C7A
@@
 $EndComp
 $Comp
-L Electronics:DRV8243 U?
-U 1 1 6160C88E
-P 2300 2250
-F 0 "U?" H 2000 2850 50  0000 C CNN
-F 1 "DRV8243" H 2500 2850 50  0000 C CNN
-F 2 "Electronics:VQFN-HR-14" H 1450 2800 50  0001 C CNN
-F 3 "https://www.ti.com/lit/ds/symlink/drv8243-q1.pdf" H 2200 2400 50  0001 C CNN
-	1    2300 2250
-	1    0    0    -1
-$EndComp
-$Comp
 L power:Earth #PWR0132
 U 1 1 616EF01B
@@
 Text Notes 10550 7650 0    50   ~ 0
 1.0
+$Comp
+L Device:R R?
+U 1 1 617496D9
+P 1350 2600
+AR Path="/615F51F3/617496D9" Ref="R?"  Part="1"
+AR Path="/617B7795/617496D9" Ref="R?"  Part="1"
+AR Path="/615F228F/617496D9" Ref="R?"  Part="1"
+F 0 "R?" H 1420 2554 50  0000 L CNN
+F 1 "100k" H 1420 2645 50  0000 L CNN
+F 2 "" V 1280 2600 50  0001 C CNN
+F 3 "~" H 1350 2600 50  0001 C CNN
+	1    1350 2600
+	-1   0    0    1
+$EndComp
+$Comp
+L Device:R R?
+U 1 1 617548F3
+P 2750 2900
+AR Path="/615F51F3/617548F3" Ref="R?"  Part="1"
+AR Path="/617B7795/617548F3" Ref="R?"  Part="1"
+AR Path="/615F228F/617548F3" Ref="R?"  Part="1"
+F 0 "R?" H 2680 2854 50  0000 R CNN
+F 1 "2.7k" H 2680 2945 50  0000 R CNN
+F 2 "" V 2680 2900 50  0001 C CNN
+F 3 "~" H 2750 2900 50  0001 C CNN
+	1    2750 2900
+	-1   0    0    1
+$EndComp
+$Comp
+L Electronics:DRV8243 U?
+U 1 1 6160C88E
+P 2300 2250
+F 0 "U?" H 2000 2850 50  0000 C CNN
+F 1 "DRV8243" H 2500 2850 50  0000 C CNN
+F 2 "Electronics:VQFN-HR-14" H 1450 2800 50  0001 C CNN
+F 3 "https://www.ti.com/lit/ds/symlink/drv8243-q1.pdf" H 2200 2400 50  0001 C CNN
+	1    2300 2250
+	1    0    0    -1
+$EndComp
+$Comp
+L Device:R R?
+U 1 1 61753AF7
+P 1600 2700
+AR Path="/615F51F3/61753AF7" Ref="R?"  Part="1"
+AR Path="/617B7795/61753AF7" Ref="R?"  Part="1"
+AR Path="/615F228F/61753AF7" Ref="R?"  Part="1"
+F 0 "R?" H 1670 2654 50  0000 L CNN
+F 1 "100k" H 1670 2745 50  0000 L CNN
+F 2 "" V 1530 2700 50  0001 C CNN
+F 3 "~" H 1600 2700 50  0001 C CNN
+	1    1600 2700
+	-1   0    0    1
+$EndComp
+$Comp
+L Device:R R?
+U 1 1 6175DC92
+P 5000 2600
+AR Path="/615F51F3/6175DC92" Ref="R?"  Part="1"
+AR Path="/617B7795/6175DC92" Ref="R?"  Part="1"
+AR Path="/615F228F/6175DC92" Ref="R?"  Part="1"
+F 0 "R?" H 5070 2554 50  0000 L CNN
+F 1 "100k" H 5070 2645 50  0000 L CNN
+F 2 "" V 4930 2600 50  0001 C CNN
+F 3 "~" H 5000 2600 50  0001 C CNN
+	1    5000 2600
+	-1   0    0    1
+$EndComp
+$Comp
+L Device:R R?
+U 1 1 6175DC98
+P 5250 2700
+AR Path="/615F51F3/6175DC98" Ref="R?"  Part="1"
+AR Path="/617B7795/6175DC98" Ref="R?"  Part="1"
+AR Path="/615F228F/6175DC98" Ref="R?"  Part="1"
+F 0 "R?" H 5320 2654 50  0000 L CNN
+F 1 "100k" H 5320 2745 50  0000 L CNN
+F 2 "" V 5180 2700 50  0001 C CNN
+F 3 "~" H 5250 2700 50  0001 C CNN
+	1    5250 2700
+	-1   0    0    1
+$EndComp
+$Comp
+L Device:R R?
+U 1 1 6175F3BD
+P 8450 2600
+AR Path="/615F51F3/6175F3BD" Ref="R?"  Part="1"
+AR Path="/617B7795/6175F3BD" Ref="R?"  Part="1"
+AR Path="/615F228F/6175F3BD" Ref="R?"  Part="1"
+F 0 "R?" H 8520 2554 50  0000 L CNN
+F 1 "100k" H 8520 2645 50  0000 L CNN
+F 2 "" V 8380 2600 50  0001 C CNN
+F 3 "~" H 8450 2600 50  0001 C CNN
+	1    8450 2600
+	-1   0    0    1
+$EndComp
+$Comp
+L Device:R R?
+U 1 1 6175F3C3
+P 8700 2700
+AR Path="/615F51F3/6175F3C3" Ref="R?"  Part="1"
+AR Path="/617B7795/6175F3C3" Ref="R?"  Part="1"
+AR Path="/615F228F/6175F3C3" Ref="R?"  Part="1"
+F 0 "R?" H 8770 2654 50  0000 L CNN
+F 1 "100k" H 8770 2745 50  0000 L CNN
+F 2 "" V 8630 2700 50  0001 C CNN
+F 3 "~" H 8700 2700 50  0001 C CNN
+	1    8700 2700
+	-1   0    0    1
+$EndComp
+$Comp
+L Device:R R?
+U 1 1 6176235A
+P 6400 2900
+AR Path="/615F51F3/6176235A" Ref="R?"  Part="1"
+AR Path="/617B7795/6176235A" Ref="R?"  Part="1"
+AR Path="/615F228F/6176235A" Ref="R?"  Part="1"
+F 0 "R?" H 6330 2854 50  0000 R CNN
+F 1 "2.7k" H 6330 2945 50  0000 R CNN
+F 2 "" V 6330 2900 50  0001 C CNN
+F 3 "~" H 6400 2900 50  0001 C CNN
+	1    6400 2900
+	-1   0    0    1
+$EndComp
+$Comp
+L Device:R R?
+U 1 1 61764625
+P 9850 2900
+AR Path="/615F51F3/61764625" Ref="R?"  Part="1"
+AR Path="/617B7795/61764625" Ref="R?"  Part="1"
+AR Path="/615F228F/61764625" Ref="R?"  Part="1"
+F 0 "R?" H 9780 2854 50  0000 R CNN
+F 1 "2.7k" H 9780 2945 50  0000 R CNN
+F 2 "" V 9780 2900 50  0001 C CNN
+F 3 "~" H 9850 2900 50  0001 C CNN
+	1    9850 2900
+	-1   0    0    1
+$EndComp
 $EndSCHEMATC

Commit message: Various fixes, added ESD protection
Parts:
- C? (x3): value 4.7uF -> 47uF
Changed lines of the file:
@@
 P 2600 1100
 F 0 "C?" V 2855 1100 50  0000 C CNN
-F 1 "4.7uF" V 2764 1100 50  0000 C CNN
+F 1 "47uF" V 2764 1100 50  0000 C CNN
 F 2 "" H 2638 950 50  0001 C CNN
 F 3 "~" H 2600 1100 50  0001 C CNN
@@
 P 6250 1100
 F 0 "C?" V 6505 1100 50  0000 C CNN
-F 1 "4.7uF" V 6414 1100 50  0000 C CNN
+F 1 "47uF" V 6414 1100 50  0000 C CNN
 F 2 "" H 6288 950 50  0001 C CNN
 F 3 "~" H 6250 1100 50  0001 C CNN
@@
 P 9700 1100
 F 0 "C?" V 9955 1100 50  0000 C CNN
-F 1 "4.7uF" V 9864 1100 50  0000 C CNN
+F 1 "47uF" V 9864 1100 50  0000 C CNN
 F 2 "" H 9738 950 50  0001 C CNN
 F 3 "~" H 9700 1100 50  0001 C CNN

Commit message: Updated rev numbers
Other:
- note added: "1.1"
- note added: "24/10/2021"
- note removed: "1.0"
- note removed: "21/10/2021"
Changed lines of the file:
@@
 Kurkkumopo HBridge driver
 Text Notes 8100 7650 0    50   ~ 0
-21/10/2021
+24/10/2021
 Text Notes 10550 7650 0    50   ~ 0
-1.0
+1.1
 $Comp
 L Device:R R?
