File: electronics/Electronics.sch (KiCad schematic (older format))
At the start: 26 parts, among them U1 STM32G441KBT3, U2 MAX14930DASE+, U3 MAX14930DASE+, U4 MAX14930DASE+

Commit message: Spurdo v2.1 update
Parts:
- added C32: 0.1uF, Capacitor_SMD:C_0603_1608Metric_Pad1.08x0.95mm_HandSolder, symbol Device:C
Connections:
- wire segments 124 -> 126
Changed lines of the file:
@@
 Text Label 700  2950 0    50   ~ 0
 MCU-debug-LED_R1
+Text Label 700  2450 0    50   ~ 0
+MCU-debug-LED_G2
 Text Label 700  2350 0    50   ~ 0
-MCU-debug-LED_G2
-Text Label 700  2250 0    50   ~ 0
 MCU-debug-LED_G1
 Wire Wire Line
@@
 Wire Wire Line
 	1700 2350 700  2350
-Wire Wire Line
-	700  2250 1700 2250
 Wire Wire Line
 	1700 3450 1700 3550
@@
 Text Label 5150 3150 2    50   ~ 0
 MCU-USB_DM
-Text Label 700  2450 0    50   ~ 0
+Text Label 700  2250 0    50   ~ 0
 MCU_NRST
 Wire Wire Line
@@
 	1    0    0    -1
 $EndComp
+$Comp
+L Device:C C?
+U 1 1 61987BE0
+P 1350 2000
+AR Path="/613FDA12/61987BE0" Ref="C?"  Part="1"
+AR Path="/61987BE0" Ref="C32"  Part="1"
+F 0 "C32" V 1098 2000 50  0000 C CNN
+F 1 "0.1uF" V 1189 2000 50  0000 C CNN
+F 2 "Capacitor_SMD:C_0603_1608Metric_Pad1.08x0.95mm_HandSolder" H 1388 1850 50  0001 C CNN
+F 3 "~" H 1350 2000 50  0001 C CNN
+	1    1350 2000
+	0    1    1    0
+$EndComp
+$Comp
+L power:GND #PWR?
+U 1 1 61987BE6
+P 1200 2000
+AR Path="/613FDA12/61987BE6" Ref="#PWR?"  Part="1"
+AR Path="/61987BE6" Ref="#PWR0189"  Part="1"
+F 0 "#PWR0189" H 1200 1750 50  0001 C CNN
+F 1 "GND" H 1205 1827 50  0000 C CNN
+F 2 "" H 1200 2000 50  0001 C CNN
+F 3 "" H 1200 2000 50  0001 C CNN
+	1    1200 2000
+	1    0    0    -1
+$EndComp
+Wire Wire Line
+	700  2250 1500 2250
+Wire Wire Line
+	1500 2000 1500 2250
+Connection ~ 1500 2250
+Wire Wire Line
+	1500 2250 1700 2250
 $EndSCHEMATC
